File: ADS1292RIPBS/ads1292r.kicad_pcb (KiCad board)
At the start: 2 copper layers, 35.7 x 27.5 mm, 40 parts, among them IC1 ADS1292RIPBS, J1 Conn_01x10_Male, J2 Conn_01x04_Male, J3 Conn_01x02_Male, U1 TLV7163318PDPQR

Commit message: v0.2
Parts:
- added G***: LOGO, udlabs:udlabs_21.1x4.4_fs, B.Cu at (142.2, 81.4)
- added G***: LOGO, udlabs:udlabs_torso_2lead_ECG, B.Cu at (138.4, 96.1)
- added G***: LOGO, udlabs:udlabs_6.0x4.5_LOGO_fs, F.Cu at (134.9, 89.9)
- added REF**: OSHW-Logo2_7.3x6mm_SilkScreen, Symbol:OSHW-Logo2_7.3x6mm_SilkScreen, B.Cu at (148.5, 95.5)
Routing:
- net DVDD: track 43.4 -> 42.7 mm
Other:
- board text added: "ADS1292R 2ch ECG + 1ch Resp."
- board text added: "DEC 2020"
- board text added: "GPIO1"
- board text added: "GPIO2"
- board text added: "MISO"
- board text added: "MOSI"
- board text removed: "DIN"
- board text removed: "DOUT"
